Commit message: Added gripper to UR5. Add .gitignore, update model URIs, remove unused model.config files, and implement gripper controller script

File: models/desk.urdf (robot description, URDF)
Before this commit: robot tavolo, 1 links, 0 joints
Links:
- link link: geometry collision box size=1 0.15 0.15; collision box size=1 0.8 0.04

File: models/ur_gz.urdf.xacro (robot description, xacro)
@@ -5,4 +5,5 @@
   <!-- import main macro -->
   <xacro:include filename="$(find ur_description)/urdf/ur_macro.xacro"/>
+  <xacro:include filename="soft_robotics_gripper.xacro"/>
   <xacro:include filename="$(find ros2_ur5_interface)/models/ur_gz.ros2_control.xacro" />
   <!-- possible 'ur_type' values: ur3, ur3e, ur5, ur5e, ur10, ur10e, ur16e, ur20, ur30 -->
@@ -38,4 +39,11 @@
     <origin xyz="0 0 0" rpy="0 0 0" />          <!-- position robot in the world -->
   </xacro:ur_robot>
+  <!-- gripper -->
+   <xacro:soft_robotics_gripper
+     parent="tool0"
+     prefix=""
+     >
+     <origin xyz="0 0 0" rpy="0 0 0" />          <!-- position robot in the world -->
+   </xacro:soft_robotics_gripper>
   <gazebo reference="world">
   </gazebo>
