Commit message: Refactor model configurations: rename and update model files, modify author details, and enhance camera and block definitions

File: models/desk.urdf.xacro (robot description, xacro)
@@ -1,15 +1,15 @@
 <?xml version="1.0" ?>
-<robot name="tavolo" xmlns:xacro="http://www.ros.org/wiki/xacro">
+<robot name="desk" xmlns:xacro="http://www.ros.org/wiki/xacro">
   <!-- Static property -->
-  <link name="link">
+  <link name="desk">
     <!-- Base collision -->
-    <collision name="base">
-      <origin xyz="0.5 0.4 0.85" rpy="0 0 0" />
+    <collision name="desk_base">
+      <origin xyz="0.5 0.4 0.435" rpy="0 0 0" />
       <geometry>
-        <box size="1 0.8 0.04" />
+        <box size="1 0.8 0.87" />
       </geometry>
     </collision>
     <!-- Box collision -->
-    <collision name="box">
+    <collision name="desk_box">
       <origin xyz="0.5 0.08 0.95" rpy="0 0 0" />
       <geometry>
@@ -18,5 +18,5 @@
     </collision>
     <!-- Back collision -->
-    <collision name="back">
+    <collision name="desk_back">
       <origin xyz="0.5 -0.02 1.35" rpy="1.57 0 0" />
       <geometry>
@@ -28,5 +28,5 @@
       <origin xyz="0 0 0" rpy="0 0 0" />
       <geometry>
-        <mesh filename="package://ros2_ur5_interface/models/meshes/desk.stl" scale="0.001 0.001 0.001" />
+        <mesh filename="file://$(find ros2_ur5_interface)/models/meshes/desk.stl" scale="0.001 0.001 0.001" />
       </geometry>
       <material name="grey_material">

File: models/ur_gz.urdf.xacro (robot description, xacro)
@@ -6,4 +6,5 @@
   <xacro:include filename="$(find ur_description)/urdf/ur_macro.xacro"/>
   <xacro:include filename="soft_robotics_gripper.xacro"/>
+  <xacro:include filename="$(find ros2_ur5_interface)/models/desk.urdf.xacro" />
   <xacro:include filename="$(find ros2_ur5_interface)/models/ur_gz.ros2_control.xacro" />
   <!-- possible 'ur_type' values: ur3, ur3e, ur5, ur5e, ur10, ur10e, ur16e, ur20, ur30 -->
@@ -21,11 +22,9 @@
   <xacro:arg name="safety_k_position" default="20"/>
   <xacro:arg name="simulation_controllers" default="" />
-  <!-- create link fixed to the "world" -->
-  <link name="world" />
   <!-- arm -->
   <xacro:ur_robot
     name="$(arg name)"
     tf_prefix="$(arg tf_prefix)"
-    parent="world"
+    parent="desk"
     joint_limits_parameters_file="$(arg joint_limit_params)"
     kinematics_parameters_file="$(arg kinematics_params)"
@@ -37,5 +36,5 @@
     force_abs_paths="true"
     >
-    <origin xyz="0 0 0" rpy="0 0 0" />          <!-- position robot in the world -->
+    <origin xyz="0.50 0.34 1.79" rpy="0 3.1415 0" />          <!-- position robot in the desk -->
   </xacro:ur_robot>
   <!-- gripper -->
@@ -44,7 +43,7 @@
      prefix=""
      >
-     <origin xyz="0 0 0" rpy="0 0 0" />          <!-- position robot in the world -->
+     <origin xyz="0 0 0" rpy="0 0 0" />          <!-- position robot in the desk -->
    </xacro:soft_robotics_gripper>
-  <gazebo reference="world">
+  <gazebo reference="desk">
   </gazebo>
   <gazebo>
