Commit message: Add gripper controller and update camera settings: include std_srvs dependency, adjust camera update rate, and configure gripper parameters in UR controllers

File: models/soft_robotics_gripper.xacro (robot description, xacro)
@@ -33,9 +33,10 @@
       </inertial>
     </link>
-    <joint name="${prefix}soft_robotics_gripper_left_finger_joint1" type="fixed">
+    <joint name="${prefix}soft_robotics_gripper_left_finger_joint1" type="revolute">
       <origin xyz="0 -0.028 0.09" rpy=" 0 0 0" />
       <parent link="${prefix}soft_robotics_gripper_base_link" />
       <child link="${prefix}soft_robotics_left_finger_link1" />
-      <limit effort="1" velocity="1" lower="-0.30" upper="0" />
+      <limit effort="1" velocity="1" lower="-0.30" upper="0.30" />
+      <axis xyz="1 0 0"/>
     </joint>
     <link name="${prefix}soft_robotics_left_finger_link1">
@@ -59,9 +60,10 @@
       </inertial>
     </link>
-    <joint name="${prefix}soft_robotics_gripper_right_finger_joint1" type="fixed">
+    <joint name="${prefix}soft_robotics_gripper_right_finger_joint1" type="revolute">
       <origin xyz="0 0.028 0.09" rpy=" 0 0 ${-pi}" />
       <parent link="${prefix}soft_robotics_gripper_base_link" />
       <child link="${prefix}soft_robotics_right_finger_link1" />
-      <limit effort="1" velocity="1" lower="-0.30" upper="0" />
+      <limit effort="1" velocity="1" lower="-0.30" upper="0.30" />
+      <axis xyz="1 0 0"/>
     </joint>
     <link name="${prefix}soft_robotics_right_finger_link1">
@@ -131,19 +133,52 @@
       </inertial>
     </link>
-  <gazebo reference="${prefix}soft_robotics_gripper_base_link">
+    <gazebo reference="${prefix}soft_robotics_gripper_base_link">
         <material>Gazebo/Grey</material>
-  </gazebo>
-  <gazebo reference="${prefix}soft_robotics_left_finger_link1">
-        <material>Gazebo/Blue</material>
-  </gazebo>
-  <gazebo reference="${prefix}soft_robotics_right_finger_link1">
-        <material>Gazebo/Blue</material>
-  </gazebo>
-    <gazebo reference="${prefix}soft_robotics_left_finger_link2">
-        <material>Gazebo/Blue</material>
-  </gazebo>
-  <gazebo reference="${prefix}soft_robotics_right_finger_link2">
-        <material>Gazebo/Blue</material>
-  </gazebo>
+    </gazebo>
+    <gazebo reference="${prefix}soft_robotics_left_finger_link1">
+        <material>Gazebo/Blue</material>
+    </gazebo>
+    <gazebo reference="${prefix}soft_robotics_right_finger_link1">
+        <material>Gazebo/Blue</material>
+    </gazebo>
+      <gazebo reference="${prefix}soft_robotics_left_finger_link2">
+        <material>Gazebo/Blue</material>
+    </gazebo>
+    <gazebo reference="${prefix}soft_robotics_right_finger_link2">
+        <material>Gazebo/Blue</material>
+    </gazebo>
+    <ros2_control name="gripper" type="system">
+        <hardware>
+          <plugin>gz_ros2_control/GazeboSimSystem</plugin>
+        </hardware>
+        <joint name="${prefix}soft_robotics_gripper_left_finger_joint1">
+          <command_interface name="position"/>
+          <command_interface name="velocity"/>
+          <state_interface name="position">
+            <!-- initial position for the mock system and simulation -->
+            <param name="initial_value">0.0</param>
+          </state_interface>
+          <state_interface name="velocity">
+            <param name="initial_value">0.0</param>
+          </state_interface>
+          <state_interface name="effort">
+            <param name="initial_value">0.0</param>
+          </state_interface>
+        </joint>
+        <joint name="${prefix}soft_robotics_gripper_right_finger_joint1">
+          <command_interface name="position"/>
+          <command_interface name="velocity"/>
+          <state_interface name="position">
+            <!-- initial position for the mock system and simulation -->
+            <param name="initial_value">0.0</param>
+          </state_interface>
+          <state_interface name="velocity">
+            <param name="initial_value">0.0</param>
+          </state_interface>
+          <state_interface name="effort">
+            <param name="initial_value">0.0</param>
+          </state_interface>
+        </joint>
+    </ros2_control>
     <!-- TRANSMISSION -->
     <transmission name="${prefix}right_finger_trans">

Commit message: Update gripper limits to avoid stucked fingers and clean up debug output in gripper service

File: models/soft_robotics_gripper.xacro (robot description, xacro)
@@ -37,5 +37,5 @@
       <parent link="${prefix}soft_robotics_gripper_base_link" />
       <child link="${prefix}soft_robotics_left_finger_link1" />
-      <limit effort="1" velocity="1" lower="-0.30" upper="0.30" />
+      <limit effort="1" velocity="1" lower="-0.35" upper="0.35" />
       <axis xyz="1 0 0"/>
     </joint>
@@ -64,5 +64,5 @@
       <parent link="${prefix}soft_robotics_gripper_base_link" />
       <child link="${prefix}soft_robotics_right_finger_link1" />
-      <limit effort="1" velocity="1" lower="-0.30" upper="0.30" />
+      <limit effort="1" velocity="1" lower="-0.35" upper="0.35" />
       <axis xyz="1 0 0"/>
     </joint>
