Commit message: Refactor simulation launch: adjust desk and camera spawn parameters, add desk state publisher, and activate gripper service

File: models/ur_gz.urdf.xacro (robot description, xacro)
@@ -6,5 +6,4 @@
   <xacro:include filename="$(find ur_description)/urdf/ur_macro.xacro"/>
   <xacro:include filename="soft_robotics_gripper.xacro"/>
-  <xacro:include filename="$(find ros2_ur5_interface)/models/desk.urdf.xacro" />
   <xacro:include filename="$(find ros2_ur5_interface)/models/ur_gz.ros2_control.xacro" />
   <!-- possible 'ur_type' values: ur3, ur3e, ur5, ur5e, ur10, ur10e, ur16e, ur20, ur30 -->
@@ -22,4 +21,11 @@
   <xacro:arg name="safety_k_position" default="20"/>
   <xacro:arg name="simulation_controllers" default="" />
+  <link name="desk">
+    <collision>
+      <geometry>
+        <box size="1.0 1.0 0.0001"/>
+      </geometry>
+    </collision>
+  </link>
   <!-- arm -->
   <xacro:ur_robot
@@ -45,6 +51,4 @@
      <origin xyz="0 0 0" rpy="0 0 0" />          <!-- position robot in the desk -->
    </xacro:soft_robotics_gripper>
-  <gazebo reference="desk">
-  </gazebo>
   <gazebo>
     <plugin filename="gz_ros2_control-system" name="gz_ros2_control::GazeboSimROS2ControlPlugin">
