Commit message: Enhance simulation launch: add multiple block types, introduce desk model with inertial properties, and adjust camera update rate

File: models/block.urdf.xacro (robot description, xacro)
@@ -37,7 +37,8 @@
       <!-- Collision Properties -->
       <collision>
-        <origin xyz="0 0 0.0285" rpy="0 0 0" />
+        <origin xyz="0 0 0" rpy="0 0 0" />
         <geometry>
-          <box size="0.031 0.031 0.057" />
+          <!-- <box size="0.031 0.031 0.057" /> -->
+          <mesh filename="file://${mesh_path}" scale="1 1 1" />
         </geometry>
       </collision>

File: models/desk.urdf.xacro (robot description, xacro)
@@ -3,4 +3,10 @@
   <!-- Static property -->
   <link name="desk">
+    <!-- Inertial -->
+    <inertial>
+      <origin xyz="0.5 0.4 0.435" rpy="0 0 0" />
+      <mass value="10" />
+      <inertia ixx="0.1" ixy="0" ixz="0" iyy="0.1" iyz="0" izz="0.1" />
+    </inertial>
     <!-- Base collision -->
     <collision name="desk_base">

Commit message: Update

File: models/block.urdf.xacro (robot description, xacro)
@@ -1,43 +1,47 @@
 <?xml version="1.0"?>
 <robot name="block" xmlns:xacro="http://ros.org/wiki/xacro">
+  <!-- Define arguments with default values -->
   <xacro:arg name="block_number" default="1" />
   <xacro:arg name="block_type" default="X1-Y1-Z2" />
-  <xacro:macro name="block" params="block_number block_type">
+  <xacro:arg name="color_input" default="0.4 0.4 0.9 1"/>
+  <xacro:arg name="px" default="0.0" />
+  <xacro:arg name="py" default="0.0" />
+  <xacro:arg name="pz" default="0.0" />
+  <xacro:arg name="ar" default="0.0" />
+  <xacro:arg name="ap" default="0.0" />
+  <xacro:arg name="ay" default="0.0" />
+  <!-- Macro definition with block_number, block_type, color_input, and other parameters -->
+  <xacro:macro name="block" params="block_number block_type color_input px py pz ar ap ay">
     <!-- Parameters for reusability -->
     <xacro:property name="mesh_path" value="$(find ros2_ur5_interface)/models/meshes/${block_type}.stl" />
     <xacro:property name="mass" value="0.01" />
-    <xacro:property name="ixx" value="3.604e-6" />
-    <xacro:property name="iyy" value="3.604e-6" />
-    <xacro:property name="izz" value="1.602e-6" />
-    <xacro:property name="color" value="0.4 0.4 0.9 1" />
     <!-- Link Definition -->
     <link name="block${block_number}">
       <!-- Inertial Properties -->
       <inertial>
-        <origin xyz="0 0 0.0285" rpy="0 0 0"/>
+        <origin xyz="0 0 0" rpy="0 0 0"/>
         <mass value="${mass}" />
         <inertia
-          ixx="${ixx}"
+          ixx="${px}"
           ixy="0"
           ixz="0"
-          iyy="${iyy}"
+          iyy="${py}"
           iyz="0"
-          izz="${izz}" />
+          izz="${pz}" />
       </inertial>
       <!-- Visual Properties -->
       <visual>
-        <origin xyz="0 0 0" rpy="0 0 0" />
+        <origin xyz="${px} ${py} ${pz}" rpy="${ar} ${ap} ${ay}" />
         <geometry>
           <mesh filename="file://${mesh_path}" scale="1 1 1" />
         </geometry>
         <material name="color">
-          <color rgba="${color}" />
+          <color rgba="${color_input}" />  <!-- Using color_input to set color -->
         </material>
       </visual>
       <!-- Collision Properties -->
       <collision>
-        <origin xyz="0 0 0" rpy="0 0 0" />
+        <origin xyz="${px} ${py} ${pz}" rpy="${ar} ${ap} ${ay}" />
         <geometry>
-          <!-- <box size="0.031 0.031 0.057" /> -->
           <mesh filename="file://${mesh_path}" scale="1 1 1" />
         </geometry>
@@ -45,4 +49,14 @@
     </link>
   </xacro:macro>
-  <xacro:block block_number="$(arg block_number)" block_type="$(arg block_type)" />
+  <!-- Instantiating the block macro with all parameters passed correctly -->
+  <xacro:block
+    block_number="$(arg block_number)"
+    block_type="$(arg block_type)"
+    color_input="$(arg color_input)"
+    px="$(arg px)"
+    py="$(arg py)"
+    pz="$(arg pz)"
+    ar="$(arg ar)"
+    ap="$(arg ap)"
+    ay="$(arg ay)" />
 </robot>

Commit message: Spawner

File: models/block.urdf.xacro (robot description, xacro)
@@ -5,34 +5,67 @@
   <xacro:arg name="block_type" default="X1-Y1-Z2" />
   <xacro:arg name="color_input" default="0.4 0.4 0.9 1"/>
-  <xacro:arg name="px" default="0.0" />
-  <xacro:arg name="py" default="0.0" />
-  <xacro:arg name="pz" default="0.0" />
-  <xacro:arg name="ar" default="0.0" />
-  <xacro:arg name="ap" default="0.0" />
-  <xacro:arg name="ay" default="0.0" />
   <!-- Macro definition with block_number, block_type, color_input, and other parameters -->
-  <xacro:macro name="block" params="block_number block_type color_input px py pz ar ap ay">
+  <xacro:macro name="block" params="block_number block_type color_input">
     <!-- Parameters for reusability -->
     <xacro:property name="mesh_path" value="$(find ros2_ur5_interface)/models/meshes/${block_type}.stl" />
     <xacro:property name="mass" value="0.01" />
+    <xacro:property name="ixx" value="3.604e-6" />
+    <xacro:property name="iyy" value="3.604e-6" />
+    <xacro:property name="izz" value="1.602e-6" />
+    <xacro:property name="scale" value="1 1 1" />
+    <!--
+  <xacro:if value="${block_type == 'X1-Y1-Z2'}">
+    <xacro:property name="scale" value="1 1 2" />
+  </xacro:if>
+  <xacro:if value="${block_type == 'X1-Y2-Z2'}">
+    <xacro:property name="scale" value="1 2 2" />
+  </xacro:if>
+  <xacro:if value="${block_type == 'X1-Y4-Z2'}">
+    <xacro:property name="scale" value="1 4 2" />
+  </xacro:if>
+  <xacro:if value="${block_type == 'X1-Y2-Z1'}">
+    <xacro:property name="scale" value="1 2 1" />
+  </xacro:if>
+  <xacro:if value="${block_type == 'X1-Y3-Z2-FILLET'}">
+    <xacro:property name="scale" value="1 3 2" />
+  </xacro:if>
+  <xacro:if value="${block_type == 'X2-Y2-Z2-FILLET'}">
+    <xacro:property name="scale" value="2 2 2" />
+  </xacro:if>
+  <xacro:if value="${block_type == 'X1-Y2-Z2-CHAMFER'}">
+    <xacro:property name="scale" value="1 2 2" />
+  </xacro:if>
+  <xacro:if value="${block_type == 'X1-Y3-Z2'}">
+    <xacro:property name="scale" value="1 3 2" />
+  </xacro:if>
+  <xacro:if value="${block_type == 'X2-Y2-Z2'}">
+    <xacro:property name="scale" value="2 2 2" />
+  </xacro:if>
+  <xacro:if value="${block_type == 'X1-Y2-Z2-TWINFILLET'}">
+    <xacro:property name="scale" value="1 2 2" />
+  </xacro:if>
+  <xacro:if value="${block_type == 'X1-Y4-Z1'}">
+    <xacro:property name="scale" value="1 4 1" />
+  </xacro:if>
+-->
     <!-- Link Definition -->
     <link name="block${block_number}">
       <!-- Inertial Properties -->
       <inertial>
-        <origin xyz="0 0 0" rpy="0 0 0"/>
+        <origin xyz="0 0 0.0285" rpy="0 0 0"/>
         <mass value="${mass}" />
         <inertia
-          ixx="${px}"
+          ixx="3.604e-6"
           ixy="0"
           ixz="0"
-          iyy="${py}"
+          iyy="3.604e-6"
           iyz="0"
-          izz="${pz}" />
+          izz="1.602e-6" />
       </inertial>
       <!-- Visual Properties -->
       <visual>
-        <origin xyz="${px} ${py} ${pz}" rpy="${ar} ${ap} ${ay}" />
+        <origin xyz="0 0 0" rpy="0 0 0" />
         <geometry>
-          <mesh filename="file://${mesh_path}" scale="1 1 1" />
+          <mesh filename="file://${mesh_path}" scale="${scale}" />
         </geometry>
         <material name="color">
@@ -42,7 +75,7 @@
       <!-- Collision Properties -->
       <collision>
-        <origin xyz="${px} ${py} ${pz}" rpy="${ar} ${ap} ${ay}" />
+        <origin xyz="0 0 0" rpy="0 0 0" />
         <geometry>
-          <mesh filename="file://${mesh_path}" scale="1 1 1" />
+          <mesh filename="file://${mesh_path}" scale="${scale}" />
         </geometry>
       </collision>
@@ -54,9 +87,4 @@
     block_type="$(arg block_type)"
     color_input="$(arg color_input)"
-    px="$(arg px)"
-    py="$(arg py)"
-    pz="$(arg pz)"
-    ar="$(arg ar)"
-    ap="$(arg ap)"
-    ay="$(arg ay)" />
+    />
 </robot>
